Commit message: 細かいところを修正

File: ws_colcon/src/my_robot_arm_description/urdf/robot.urdf.xacro (robot description, xacro)
@@ -11,9 +11,17 @@
         <color rgba="0.2 0.8 0.2 1.0"/>
     </material>
+    <!-- World Link -->
+    <link name="world"/>
+    <!-- Fixed joint between world and base_link -->
+    <joint name="world_joint" type="fixed">
+        <parent link="world"/>
+        <child link="base_link"/>
+        <origin xyz="0 0 0" rpy="0 0 0"/>
+    </joint>
     <!-- Base Link -->
     <link name="base_link">
         <visual>
             <geometry>
-                <cylinder length="0.05" radius="0.1"/>
+                <cylinder length="0.05" radius="0.06"/>
             </geometry>
             <material name="blue"/>
@@ -21,5 +29,5 @@
         <collision>
             <geometry>
-                <cylinder length="0.05" radius="0.1"/>
+                <cylinder length="0.05" radius="0.06"/>
             </geometry>
         </collision>
@@ -29,12 +37,17 @@
         <parent link="base_link"/>
         <child link="link1"/>
-        <origin xyz="0 0 0.025" rpy="0 0 0"/>
+        <origin xyz="0 0 0.05" rpy="0 0 0"/>
         <axis xyz="0 0 1"/>
         <limit lower="-2.356" upper="2.356" effort="100" velocity="1"/>  <!-- -135° to +135° -->
     </joint>
     <link name="link1">
+        <inertial>
+            <origin xyz="0 0 0.075" rpy="0 0 0"/>
+            <mass value="0.5"/>
+            <inertia ixx="0.002" ixy="0" ixz="0" iyy="0.002" iyz="0" izz="0.001"/>
+        </inertial>
         <visual>
             <geometry>
-                <cylinder length="0.05" radius="0.05"/>
+                <cylinder length="0.15" radius="0.03"/>
             </geometry>
             <material name="red"/>
@@ -42,5 +55,5 @@
         <collision>
             <geometry>
-                <cylinder length="0.05" radius="0.05"/>
+                <cylinder length="0.15" radius="0.03"/>
             </geometry>
         </collision>
@@ -50,12 +63,17 @@
         <parent link="link1"/>
         <child link="link2"/>
-        <origin xyz="0 0 0.05" rpy="0 0 0"/>
+        <origin xyz="0 0 0.15" rpy="0 0 0"/>
         <axis xyz="1 0 0"/>
         <limit lower="-2.356" upper="2.356" effort="100" velocity="1"/>  <!-- -135° to +135° -->
     </joint>
     <link name="link2">
+        <inertial>
+            <origin xyz="0 0 0.03" rpy="0 0 0"/>
+            <mass value="0.3"/>
+            <inertia ixx="0.0005" ixy="0" ixz="0" iyy="0.0005" iyz="0" izz="0.0001"/>
+        </inertial>
         <visual>
             <geometry>
-                <box size="0.05 0.05 0.15"/>
+                <box size="0.03 0.03 0.06"/>
             </geometry>
             <material name="green"/>
@@ -63,5 +81,5 @@
         <collision>
             <geometry>
-                <box size="0.05 0.05 0.15"/>
+                <box size="0.03 0.03 0.06"/>
             </geometry>
         </collision>
@@ -71,12 +89,17 @@
         <parent link="link2"/>
         <child link="link3"/>
-        <origin xyz="0 0 0.15" rpy="0 0 0"/>
+        <origin xyz="0 0.02 0.1" rpy="0 0 0"/>
         <axis xyz="1 0 0"/>
         <limit lower="-2.356" upper="2.356" effort="100" velocity="1"/>  <!-- -135° to +135° -->
     </joint>
     <link name="link3">
+        <inertial>
+            <origin xyz="0 0 0.04" rpy="0 0 0"/>
+            <mass value="0.3"/>
+            <inertia ixx="0.0005" ixy="0" ixz="0" iyy="0.0005" iyz="0" izz="0.0001"/>
+        </inertial>
         <visual>
             <geometry>
-                <box size="0.05 0.05 0.15"/>
+                <box size="0.03 0.03 0.06"/>
             </geometry>
             <material name="blue"/>
@@ -84,5 +107,5 @@
         <collision>
             <geometry>
-                <box size="0.05 0.05 0.15"/>
+                <box size="0.03 0.03 0.06"/>
             </geometry>
         </collision>
@@ -92,9 +115,14 @@
         <parent link="link3"/>
         <child link="link4"/>
-        <origin xyz="0 0 0.15" rpy="0 0 0"/>
+        <origin xyz="0 0 0.06" rpy="0 0 0"/>
         <axis xyz="1 0 0"/>
         <limit lower="-2.356" upper="2.356" effort="100" velocity="1"/>  <!-- -135° to +135° -->
     </joint>
     <link name="link4">
+        <inertial>
+            <origin xyz="0 0 0.025" rpy="0 0 0"/>
+            <mass value="0.3"/>
+            <inertia ixx="0.0005" ixy="0" ixz="0" iyy="0.0005" iyz="0" izz="0.0001"/>
+        </inertial>
         <visual>
             <geometry>
@@ -118,4 +146,9 @@
     </joint>
     <link name="end_effector">
+        <inertial>
+            <origin xyz="0 0 0.025" rpy="0 0 0"/>
+            <mass value="0.1"/>
+            <inertia ixx="0.0001" ixy="0" ixz="0" iyy="0.0001" iyz="0" izz="0.0001"/>
+        </inertial>
         <visual>
             <geometry>

Commit message: 長さを伸ばす

File: ws_colcon/src/my_robot_arm_description/urdf/robot.urdf.xacro (robot description, xacro)
@@ -115,5 +115,5 @@
         <parent link="link3"/>
         <child link="link4"/>
-        <origin xyz="0 0 0.06" rpy="0 0 0"/>
+        <origin xyz="0 0 0.08" rpy="0 0 0"/>
         <axis xyz="1 0 0"/>
         <limit lower="-2.356" upper="2.356" effort="100" velocity="1"/>  <!-- -135° to +135° -->
